Commit message: calibrate camera pose

File: panda_arm_hand_camera.urdf (robot description, URDF)
Before this commit: robot panda, 13 links, 12 joints
Joints:
- joint panda_hand_camera_joint: origin xyz=0.04 0 0.03 rpy=-1.57079632679 0 -1.57079632679   -> xyz=0.036 0 0.031 rpy=-1.57079632679 0 -1.57079632679  

Commit message: cleanup files

File: panda_arm_hand_camera.urdf (robot description, URDF)
Before this commit: robot panda, 13 links, 12 joints
Joints:
- joint panda_hand_camera_joint: origin xyz=0.036 0 0.031 rpy=-1.57079632679 0 -1.57079632679   -> xyz=0.036 0 0.036 rpy=-1.57079632679 0 -1.57079632679
